File: inner/badge-inner2-revB.brd (EAGLE design)
At the start: 54 x 61 mm, 29 parts, among them J1 TC2030-CTX-NL, Q1 DMP2240UDM, U1 SKB369, U3 SN74LVC2G04

Commit message: Minor changes to layout
Parts:
- moved SW2 0.08 mm to (0.00, 11.6)
Other:
- outline, holes or cut-outs redrawn
Changed lines of the file:
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@@
 <setting verticaltext="up"/>
 </settings>
-<grid distance="5" unitdist="mil" unit="mil" style="lines" multiple="1" display="yes" altdistance="1" altunitdist="mil" altunit="mil"/>
+<grid distance="0.1" unitdist="mm" unit="mm" style="lines" multiple="1" display="yes" altdistance="1" altunitdist="mil" altunit="mil"/>
 <layers>
 <layer number="1" name="Top" color="4" fill="1" visible="yes" active="yes"/>
@@
 <attribute name="VALUE" x="51.143" y="56.27" size="0.6096" layer="27" font="vector" ratio="20" rot="R90" align="top-center"/>
 </element>
-<element name="SW2" library="shlomo" package="EVQP4KB" value="" x="0" y="11.5" smashed="yes" rot="R270"/>
+<element name="SW2" library="shlomo" package="EVQP4KB" value="" x="0" y="11.5762" smashed="yes" rot="R270"/>
 <element name="C5" library="SparkFun-Capacitors" library_urn="urn:adsk.eagle:library:510" package="0603" package3d_urn="urn:adsk.eagle:package:37414/1" value="0.1uF" x="6" y="9.5" smashed="yes">
 <attribute name="NAME" x="6" y="10.262" size="0.6096" layer="25" font="vector" ratio="20" align="bottom-center"/>
@@
 <contactref element="SW2" pad="1"/>
 <contactref element="R5" pad="1"/>
-<wire x1="2.575" y1="13.775" x2="5.15" y2="13.775" width="0.254" layer="1"/>
-<wire x1="5.15" y1="13.775" x2="5.15" y2="13.5" width="0.254" layer="1"/>
+<wire x1="2.575" y1="13.8512" x2="5.15" y2="13.8512" width="0.254" layer="1"/>
+<wire x1="5.15" y1="13.8512" x2="5.15" y2="13.5" width="0.254" layer="1"/>
 </signal>
 <signal name="SW2">
