File: outer/keycard-outer-revA.brd (EAGLE design)
At the start: 54 x 86 mm, 1 part

Commit message: Minor changes to layout
Other:
- board text added: "ALL ACCESS"
- board text removed: "MULTI PASS"
Changed lines of the file:
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@@
 <layer number="2" name="Route2" color="16" fill="1" visible="no" active="no"/>
 <layer number="15" name="Route15" color="23" fill="1" visible="no" active="no"/>
-<layer number="16" name="Bottom" color="1" fill="1" visible="no" active="yes"/>
-<layer number="17" name="Pads" color="2" fill="1" visible="no" active="yes"/>
-<layer number="18" name="Vias" color="2" fill="1" visible="no" active="yes"/>
-<layer number="19" name="Unrouted" color="6" fill="1" visible="no" active="yes"/>
-<layer number="20" name="Dimension" color="24" fill="1" visible="no" active="yes"/>
+<layer number="16" name="Bottom" color="1" fill="1" visible="yes" active="yes"/>
+<layer number="17" name="Pads" color="2" fill="1" visible="yes" active="yes"/>
+<layer number="18" name="Vias" color="2" fill="1" visible="yes" active="yes"/>
+<layer number="19" name="Unrouted" color="6" fill="1" visible="yes" active="yes"/>
+<layer number="20" name="Dimension" color="24" fill="1" visible="yes" active="yes"/>
 <layer number="21" name="tPlace" color="7" fill="1" visible="yes" active="yes"/>
 <layer number="22" name="bPlace" color="7" fill="1" visible="no" active="yes"/>
@@
 <layer number="43" name="vRestrict" color="2" fill="10" visible="no" active="yes"/>
 <layer number="44" name="Drills" color="7" fill="1" visible="no" active="yes"/>
-<layer number="45" name="Holes" color="7" fill="1" visible="no" active="yes"/>
-<layer number="46" name="Milling" color="3" fill="1" visible="no" active="yes"/>
+<layer number="45" name="Holes" color="7" fill="1" visible="yes" active="yes"/>
+<layer number="46" name="Milling" color="3" fill="1" visible="yes" active="yes"/>
 <layer number="47" name="Measures" color="7" fill="1" visible="no" active="yes"/>
 <layer number="48" name="Document" color="7" fill="1" visible="no" active="yes"/>
@@
 <vertex x="27.24743125" y="49.022209375"/>
 </polygon>
-<text x="4.953" y="4.699" size="6.858" layer="21" font="vector" ratio="10">MULTI PASS</text>
+<text x="4.953" y="4.699" size="6.858" layer="21" font="vector" ratio="10">ALL ACCESS</text>
 <wire x1="6.079" y1="7.982" x2="6.079" y2="3.907" width="0.01" layer="201"/>
 <wire x1="6.079" y1="3.907" x2="7.729" y2="3.907" width="0.01" layer="201"/>
@@
 <wire x1="41.552259375" y1="67.79681875" x2="41.182609375" y2="67.80361875" width="0.01" layer="202" curve="26.87"/>
 <wire x1="41.182609375" y1="67.80361875" x2="40.88" y2="67.638" width="0.01" layer="202" curve="32.62"/>
+<hole x="22.098" y="79.248" drill="2.54"/>
+<hole x="32.004" y="79.248" drill="2.54"/>
 </plain>
 <attributes>
